File: downstream_port.kicad_sch (KiCad schematic)
At the start: 7 parts, among them U2 MIC2026-1YM

Commit message: public release revA
Parts:
- added D4, D6: A, LED_SMD:LED_0603_1608Metric, symbol Device:LED_Filled
- added D5, D7: B, LED_SMD:LED_0603_1608Metric, symbol Device:LED_Filled
- added R49, R51: 150R, Resistor_SMD:R_0603_1608Metric, symbol Device:R_US
- added R50, R52: 680R, Resistor_SMD:R_0603_1608Metric, symbol Device:R_US
- R53: renamed from R2; footprint (none) -> Resistor_SMD:R_0603_1608Metric
- R54: renamed from R4; footprint (none) -> Resistor_SMD:R_0603_1608Metric
- U4: renamed from U2; footprint Package_DIP:DIP-8_W7.62mm -> Package_SO:SO-8_3.9x4.9mm_P1.27mm
- renumbered C1 to C27, C2 to C28, D1 to D8, D2 to D9
Connections:
- net OUTA renamed VBUS_OUTA
- net OUTB renamed VBUS_OUTB
- new net: D6.2 (A), R51.1
- new net: D5.2 (A), R50.1
- new net: D4.2 (A), R49.1
- new net: D7.2 (A), R52.1
- new net +3V3: R49.2, R50.2, R51.2, R52.2
- new net LEDA1: D4.1 (K)
- new net LEDA2: D6.1 (K)
- new net LEDB1: D5.1 (K)
- new net LEDB2: D7.1 (K)
Other:
- note added: "Dual Channel Power Distributon Switch 500mA/channel"
- note added: "LEDA LOW = LS device attached LEDA HIGH = FS device attached LEDA 1KHz = HS device attached LEDA TRI = no device attached"
- note added: "STATUS LEDs"
- company: (none) -> Voltlog
- title: (none) -> VoltHub7
- moved on the sheet: C27, C28, D8, D9, R53, R54, U4
