File: volthub7.kicad_sch (KiCad schematic)
At the start: 9 parts, among them U1 USB2517, U3 AT24C02C

Commit message: public release revA
Parts:
- removed D33, D55: ~, LED_SMD:LED_0603_1608Metric, symbol Device:LED_Filled
- removed R1: 650R, symbol Device:R_US
- removed R3: 10K, symbol Device:R_US
- removed R3: 180R, symbol Device:R_US
- added C1, C20, C21, C22, C23, C24, C25, C26: 4.7nF, Capacitor_SMD:C_1206_3216Metric, symbol Device:C
- added C10, C14, C15, C16, C19, C4, C46, C6, C8, C9: 0.1uF, Capacitor_SMD:C_0603_1608Metric, symbol Device:C
- added C11, C18, C3, C5, C7: 1uF, Capacitor_SMD:C_0603_1608Metric, symbol Device:C
- added C12, C13: 15pF, Capacitor_SMD:C_0603_1608Metric, symbol Device:C_Small
- added D1: SP0503BAHT, Package_TO_SOT_SMD:SOT-143, symbol Power_Protection:SP0503BAHT
- added D2: EEPROM, LED_SMD:LED_0603_1608Metric, symbol Device:LED_Filled
- added D3: DEFAULT, LED_SMD:LED_0603_1608Metric, symbol Device:LED_Filled
- added FID1, FID2, FID3: Fiducial, Fiducial:Fiducial_0.5mm_Mask1mm, symbol Mechanical:Fiducial
- added H1, H2, H3, H4, H5, H6, H7: MountingHole, MountingHole:MountingHole_3.2mm_M3, symbol Mechanical:MountingHole
- added H10, H11, H8, H9: M3x11mm, Voltlog:SMTSO30100CTJ, symbol Mechanical:MountingHole_Pad
- added J1: USB_B, Connector_USB:USB_B_Lumberg_2411_02_Horizontal, symbol Connector:USB_B
- added J10: USB_7, Voltlog:USB_A_HRO_U-A-24DD-W-5, symbol Connector:USB_A
- added J2: TEST JIG, Voltlog:JST_PHD_B32B-PHDSS_2x20_P2.00mm_Vertical, symbol Connector_Generic:Conn_02x20_Odd_Even
- added J3: TYPE-C-31-M-12, Voltlog:USB_C_Receptacle_HRO_TYPE-C-31-M-12, symbol Voltlog:USB_C_Receptacle_USB2.0
- added J4: USB_1, Voltlog:USB_A_HRO_U-A-24DD-W-5, symbol Connector:USB_A
- added J5: USB_2, Voltlog:USB_A_HRO_U-A-24DD-W-5, symbol Connector:USB_A
- added J6: USB_3, Voltlog:USB_A_HRO_U-A-24DD-W-5, symbol Connector:USB_A
- added J7: USB_4, Voltlog:USB_A_HRO_U-A-24DD-W-5, symbol Connector:USB_A
- added J8: USB_5, Voltlog:USB_A_HRO_U-A-24DD-W-5, symbol Connector:USB_A
- added J9: USB_6, Voltlog:USB_A_HRO_U-A-24DD-W-5, symbol Connector:USB_A
- added R1, R10, R11, R12, R13, R14, R15, R16, R17, R18, R19, R20, R21, R22, R23, R34, R35, R36, R37, R38, R39, R40, R41, R42, R43, R44, R45, R46, R47, R8, R9: 0R, Resistor_SMD:R_0603_1608Metric, symbol Device:R_Small_US
- added R2: 1M, Resistor_SMD:R_1206_3216Metric, symbol Device:R_US
- added R24, R25, R27, R28, R29: 100K, Resistor_SMD:R_0603_1608Metric, symbol Device:R_US
- added R26: 1M, Resistor_SMD:R_0603_1608Metric, symbol Device:R_US
- added R3: 0R, Resistor_SMD:R_0603_1608Metric, symbol Device:R_US
- added R30: 1K5, Resistor_SMD:R_0603_1608Metric, symbol Device:R_US
- added R31, R32, R4, R5, R98: 10K, Resistor_SMD:R_0603_1608Metric, symbol Device:R_US
- added R33: 1K, Resistor_SMD:R_0603_1608Metric, symbol Device:R_US
- added R48: 12K, Resistor_SMD:R_0603_1608Metric, symbol Device:R_US
- added R6, R7: 5K1, Resistor_SMD:R_0603_1608Metric, symbol Device:R_US
- added TP1: USBUP_DN, Voltlog:Pogo_pin_YZ87615160P-01, symbol Connector:TestPoint_Probe
- added TP2: USBUP_DP, Voltlog:Pogo_pin_YZ87615160P-01, symbol Connector:TestPoint_Probe
- added TP3: UP_VBUS, Voltlog:Pogo_pin_YZ87615160P-01, symbol Connector:TestPoint_Probe
- added TP4: GND, Voltlog:Pogo_pin_YZ87615160P-01, symbol Connector:TestPoint_Probe
- added U2: RaspberryPi GPIO 40pin, Voltlog:RaspberryPi_Zero2W_40Pin, symbol Voltlog:RaspberryPi-GPIO
- added Y1: 24MHz, Crystal:Crystal_SMD_SeikoEpson_TSX3225-4Pin_3.2x2.5mm, symbol Device:Crystal_GND24
- V1: footprint (none) -> Voltlog:voltlog_mask_5mm
- renumbered C3 to C17, U3 to U1, U1 to U3
Connections:
- net RESET_USB: now reaches C17.1
- net RESET_USB: now also U3.43 (~{RESET}), R28.1, R39.2
- net GND: now reaches C17.2
- net GND: now also U1.1 (A0), U1.2 (A1), U1.3 (A2), U1.4 (GND), U3.19 (TEST), U3.65 (VSS), C1.2, C10.2, C11.2, C12.1, C13.2, C14.2, C15.2, C16.2, C18.2, C19.2, C20.2, C21.2, C22.2, C23.2, C24.2, C25.2, C26.2, C3.2, C4.2, C46.2, C5.2, C6.2, C7.2, C8.2, C9.2, D1.1 (A), D3.1 (K), J1.4 (GND), J10.4 (GND), J2.12 (Pin_12), J2.16 (Pin_16), J2.20 (Pin_20), J2.24 (Pin_24), J2.28 (Pin_28), J2.4 (Pin_4), J2.8 (Pin_8), J3.A1 (GND), J3.A12 (GND), J3.B1 (GND), J3.B12 (GND), J4.4 (GND), J5.4 (GND), J6.4 (GND), J7.4 (GND), J8.4 (GND), J9.4 (GND), R2.2, R27.1, R29.2, R3.1, R33.1, R48.1, R6.1, R7.1, R98.1, TP4.1, U2.14 (GND), U2.20 (GND), U2.25 (GND), U2.30 (GND), U2.34 (GND), U2.39 (GND), U2.6 (GND), U2.9 (GND), Y1.2, Y1.4
- net SDA: now reaches U1.5 (SDA)
- net SDA: now also U3.40 (SDA), R4.1, R9.1
- net SCL/CFG_SEL0: now reaches U1.6 (SCL)
- net SCL/CFG_SEL0: now also U3.41 (SCL), R10.1, R5.1
- net EE_WP: now reaches U1.7 (WP)
- net EE_WP: now also R11.1, R3.2
- net at U1.8 (VCC): now also C46.1, R1.1, R4.2, R5.2
- net USB1_DN: now reaches U3.1 (USBDN1_DM)
- net USB1_DN: now also J2.9 (Pin_9), J4.2 (D-)
- net +3V3: now reaches U3.10 (VDDA33)
- net +3V3: now also U3.24 (VDD33CR), U3.46 (VDD33), U3.5 (VDDA33), U3.52 (VDDA33), U3.57 (VDDA33), U3.64 (VDD33PLL), C10.1, C14.1, C15.1, C16.1, C18.1, C19.1, C7.1, C8.1, C9.1, D2.2 (A), J2.29 (Pin_29), R1.2, R15.1, R25.1, R28.2, R31.2, R32.2, R8.1
- net USB5_DN: now reaches U3.11 (USBDN5_DM)
- net USB5_DN: now also J2.25 (Pin_25), J8.2 (D-)
- net USB5_DP: now reaches U3.12 (USBDN5_DP)
- net USB5_DP: now also J2.27 (Pin_27), J8.3 (D+)
- net CFG_SEL2: now reaches U3.13 (CFG_SEL2)
- net CFG_SEL2: now also R32.1, R33.2
- net LEDB7: now reaches U3.14 (~{LEDB7})
- net LEDA1: now reaches U3.15 (~{LEDA1}/PRT_SWP1)
- net LEDB6: now reaches U3.16 (~{LEDB6})
- net LEDA2: now reaches U3.17 (~{LEDA2}/PRT_SWP2)
- net LEDB5: now reaches U3.18 (~{LEDB5})
- net USB1_DP: now reaches U3.2 (USBDN1_DP)
- net USB1_DP: now also J2.11 (Pin_11), J4.3 (D+)
- net PRTPWR4: now reaches U3.20 (PRTPWR4)
- net PRTPWR4: now also R41.2
- net OCS4: now reaches U3.21 (OCS4_N)
- net OCS4: now also R17.1
- net OCS3: now reaches U3.22 (OCS3_N)
- net OCS3: now also R42.2
- net PRTPWR3: now reaches U3.23 (PRTPWR3)
- net PRTPWR3: now also R18.1
- net VDDCR: now reaches U3.25 (VDD18)
- net VDDCR: now also C5.1, C6.1
- net PRTPWR2: now reaches U3.26 (PRTPWR2)
- net PRTPWR2: now also R43.2
- net OCS2: now reaches U3.27 (OCS2_N)
- net OCS2: now also R19.1
- net OCS1: now reaches U3.28 (OCS1_N)
- net OCS1: now also R44.2
- net PRTPWR1: now reaches U3.29 (PRTPWR1)
- net PRTPWR1: now also R20.1
- net USB2_DN: now reaches U3.3 (USBDN2_DM)
- net USB2_DN: now also J2.13 (Pin_13), J5.2 (D-)
- net PRTPWR5: now reaches U3.30 (PRTPWR5)
- net PRTPWR5: now also R21.1
- net LEDA3: now reaches U3.31 (~{LEDA3}/PRT_SWP3)
- net LEDB4: now reaches U3.32 (~{LEDB4})
- net LEDA4: now reaches U3.33 (~{LEDA4}/PRT_SWP4)
- net LEDB3: now reaches U3.34 (~{LEDB3}/GANG_EN)
- net OCS5: now reaches U3.35 (OCS5_N)
- net OCS5: now also R45.2
- net PRTPWR7: now reaches U3.36 (PRTPWR7)
- net PRTPWR7: now also R22.1
- net OCS7: now reaches U3.37 (OCS7_N)
- net OCS7: now also R46.2
- net OCS6: now reaches U3.38 (OCS6_N)
- net OCS6: now also R23.1
- net PRTPWR6: now reaches U3.39 (PRTPWR6)
- net PRTPWR6: now also R47.2
- net USB2_DP: now reaches U3.4 (USBDN2_DP)
- net USB2_DP: now also J2.15 (Pin_15), J5.3 (D+)
- net HS_IND/CFG_SEL1: now reaches U3.42 (HS_IND/CFG_SEL1)
- net HS_IND/CFG_SEL1: now also R30.2
- net VBUS_DET: now reaches U3.44 (VBUS_DET)
- net VBUS_DET: now also R24.2, R27.2
- net LOCAL_PWR: now reaches U3.45 (SUSP_IND/LOCAL_PWR/NON_REM0)
- net LOCAL_PWR: now also R31.1
- net LEDA5: now reaches U3.47 (~{LEDA5}/PRT_SWP5)
- net LEDB2: now reaches U3.48 (~{LEDB2}/BOOST1)
- net LEDA6: now reaches U3.49 (~{LEDA6}/PRT_SWP6)
- net LEDB1: now reaches U3.50 (~{LEDB1}/BOOST0)
- net LEDA7: now reaches U3.51 (~{LEDA7}/PRT_SWP7)
- net USB6_DN: now reaches U3.53 (USBDN6_DM)
- net USB6_DN: now also J2.1 (Pin_1), J9.2 (D-)
- net USB6_DP: now reaches U3.54 (USBDN6_DP)
- net USB6_DP: now also J2.3 (Pin_3), J9.3 (D+)
- net USB7_DN: now reaches U3.55 (USBDN7_DM)
- net USB7_DN: now also J10.2 (D-), J2.5 (Pin_5)
- net USB7_DP: now reaches U3.56 (USBDN7_DP)
- net USB7_DP: now also J10.3 (D+), J2.7 (Pin_7)
- net USBUP_DP: now reaches U3.59 (USBUP_DP)
- net USBUP_DP: now also D1.4 (K), J1.3 (D+), J3.A6 (D+), J3.B6 (D+), TP2.1
- net USB3_DN: now reaches U3.6 (USBDN3_DM)
- net USB3_DN: now also J2.17 (Pin_17), J6.2 (D-)
- net XTAL2: now reaches U3.60 (XTAL2)
- net XTAL2: now also C13.1, R26.1, Y1.3
- net XTAL1: now reaches U3.61 (XTAL1/CLKIN)
- net XTAL1: now also C12.2, R26.2, Y1.1
- net VDDAPLL: now reaches U3.62 (VDD18PLL)
- net VDDAPLL: now also C3.1, C4.1
- net RBIAS: now reaches U3.63 (RBIAS)
- net RBIAS: now also R48.2
- net USB3_DP: now reaches U3.7 (USBDN3_DP)
- net USB3_DP: now also J2.19 (Pin_19), J6.3 (D+)
- net USB4_DN: now reaches U3.8 (USBDN4_DM)
- net USB4_DN: now also J2.21 (Pin_21), J7.2 (D-)
- net USB4_DP: now reaches U3.9 (USBDN4_DP)
- net USB4_DP: now also J2.23 (Pin_23), J7.3 (D+)
- new net: C20.1, J4.5 (Shield)
- new net: R11.2, U2.7 (GPIO4/GPCLK0)
- new net: R36.1, U2.8 (GPIO14/TXD)
- new net: D2.1 (K), D3.2 (A), R25.2, R29.1, R30.1
- new net: R38.1, U2.12 (GPIO18/PCM_CLK)
- new net: C26.1, J10.5 (Shield)
- new net: C24.1, J8.5 (Shield)
- new net: R10.2, U2.5 (GPIO3/SCL)
- new net: R18.2, U2.23 (GPIO11/SCLK)
- new net: R20.2, U2.31 (GPIO6)
- new net: C21.1, J5.5 (Shield)
- new net: R21.2, U2.33 (GPIO13/PWM1)
- new net: R17.2, U2.21 (GPIO9/MISO)
- new net: R37.1, U2.10 (GPIO15/RXD)
- new net: R12.2, U2.11 (GPIO17)
- new net: R13.2, U2.13 (GPIO27)
- new net: R14.2, U2.15 (GPIO22)
- new net: R39.1, U2.16 (GPIO23)
- new net: R40.1, U2.18 (GPIO24)
- new net: R16.2, U2.19 (GPIO10/MOSI)
- new net: R41.1, U2.22 (GPIO25)
- new net: R42.1, U2.24 (GPIO8/CE0)
- new net: R43.1, U2.26 (GPIO7/CE1)
- new net: R19.2, U2.29 (GPIO5)
- new net: R9.2, U2.3 (GPIO2/SDA)
- new net: R44.1, U2.32 (GPIO12/PWM0)
- new net: R22.2, U2.35 (GPIO19/PCM_FS)
- new net: R45.1, U2.36 (GPIO16)
- new net: R23.2, U2.37 (GPIO26)
- new net: R46.1, U2.38 (GPIO20/PCM_DIN)
- new net: R47.1, U2.40 (GPIO21/PCM_DOUT)
- new net: C22.1, J6.5 (Shield)
- new net: C25.1, J9.5 (Shield)
- new net: C23.1, J7.5 (Shield)
- new net +5V: J2.39 (Pin_39), R34.2, R35.2
- new net DCDC_PG: R40.2
- new net GPIO18: R38.2
- new net InputOutput/LEDY_A: J2.34 (Pin_34)
- new net InputOutput/LED_G: R12.1
- new net InputOutput/LED_R: R13.1
- new net InputOutput/LED_Y: R14.1
- new net InputOutput/OLED_SCL: J2.38 (Pin_38)
- new net InputOutput/OLED_SDA: J2.36 (Pin_36)
- new net InputOutput/OLED_VDD: J2.40 (Pin_40)
- new net InputOutput/SW1_P: J2.30 (Pin_30)
- new net InputOutput/SW2_P: J2.32 (Pin_32)
- new net InputOutput/SWITCH1: R16.1
- new net LEDG_A: J2.31 (Pin_31)
- new net LEDR_A: J2.33 (Pin_33)
- new net PI_3V3: R15.2, R8.2, U2.1 (3V3), U2.17 (3V3)
- new net PI_5V: R34.1, R35.1, U2.2 (5V), U2.4 (5V)
- new net PI_RXD: J2.37 (Pin_37), R37.2
- new net PI_TXD: J2.35 (Pin_35), R36.2
- new net Port4 down1/ENB: R98.2
- new net UP_CC1: J3.A5 (CC1), R7.2
- new net UP_CC2: J3.B5 (CC2), R6.2
- new net UP_VBUS: C11.1, D1.2 (K), J1.1 (VBUS), J3.A4 (VBUS), J3.A9 (VBUS), J3.B4 (VBUS), J3.B9 (VBUS), R24.1, TP3.1
- new net USBUP_DN: D1.3 (K), J1.2 (D-), J3.A7 (D-), J3.B7 (D-), TP1.1, U3.58 (USBUP_DM)
- new net USB_SH: C1.1, J1.5 (Shield), J3.S1 (SHIELD), R2.1
- new net VBUS1: J2.10 (Pin_10), J4.1 (VBUS)
- new net VBUS2: J2.14 (Pin_14), J5.1 (VBUS)
- new net VBUS3: J2.18 (Pin_18), J6.1 (VBUS)
- new net VBUS4: J2.22 (Pin_22), J7.1 (VBUS)
- new net VBUS5: J2.26 (Pin_26), J8.1 (VBUS)
- new net VBUS6: J2.2 (Pin_2), J9.1 (VBUS)
- new net VBUS7: J10.1 (VBUS), J2.6 (Pin_6)
- no-connect marks 0 -> 12
Other:
- sheet Port1 renamed Port1 down
- added sheet InputOutput (output.kicad_sch)
- added sheet Port2 down (downstream_port.kicad_sch)
- added sheet Port3 down (downstream_port.kicad_sch)
- added sheet Port4 down1 (downstream_port_last.kicad_sch)
- added sheet Power (power.kicad_sch)
- sheet Port1 down ports: added LEDA1, LEDA2, LEDB1, LEDB2, VBUS_OUTA, VBUS_OUTB; removed GND, OUTA, OUTB
- note added: "By default EEPROM not in use."
- note added: "DOWNSTREAM PORTS"
- note added: "OPTIONAL USB Type-B"
- note added: "PRTPWRx and OCSx signals are 3V3 so it's safe to connect to PiZero! Warning: the USB2517 will not initialize until the pizero pulls RESET_USB high."
- note added: "Pi Zero Pogo Pins and Mounting Holes"
- note added: "The pi zero mounting holes are M2.5! Mounting studs height should be increased to 12mm! Pogo pin working distance 11-12mm."
- note added: "UPSTREAM PORT"
- note added: "VOLTHUB7"
- note removed: "add fuse on the input add multiple power input options"
- moved on the sheet: C17, U1
